Commit message: simulation_launch package: - modified nav2 parameters for experiment purposes - modified  all of the launch files to enable robot model file path and world file path to be alterable in robot_bringup.launch.py (top-level launch file) - made a new robot model called alphabot2

File: simulation_launch/models/test_bot/model.urdf (robot description, URDF)
Before this commit: robot mobile_bot, 5 links, 4 joints
Links:
- added link drivewhl_l_link, mass 2; collision cylinder length=0.04 radius=0.1; visual cylinder length=0.04 radius=0.1
- added link drivewhl_r_link, mass 2; collision cylinder length=0.04 radius=0.1; visual cylinder length=0.04 radius=0.1
- link base_link: mass None -> 5; geometry collision box size=0.52 0.31 0.18; visual box size=0.52 0.31 0.18
- link front_caster: mass None -> 2; geometry collision sphere radius=0.060000000000000026; visual sphere radius=0.060000000000000026
- link imu_link: mass None -> 0.1
Joints:
- added joint drivewhl_l_joint: type continuous, parent base_link, child drivewhl_l_link, origin xyz=-0.18 0.175 -0.05 rpy=0 0 0, axis 0 1 0
- added joint drivewhl_r_joint: type continuous, parent base_link, child drivewhl_r_link, origin xyz=-0.18 -0.175 -0.05 rpy=0 0 0, axis 0 1 0
- joint base_joint: origin xyz=0 0 ${(wheel_radius+wheel_zoff)} rpy=0 0 0 -> xyz=0 0 0.15000000000000002 rpy=0 0 0
- joint caster_joint: origin xyz=${caster_xoff} 0 ${-(base_height/2)} rpy=0 0 0 -> xyz=0.18 0 -0.09 rpy=0 0 0

File: simulation_launch/models/test_bot/model.xacro (robot description, xacro)
@@ -1,13 +1,40 @@
-<?xml version="1.0" ?>
-<!-- =================================================================================== -->
-<!-- |    This document was autogenerated by xacro from xacro_model.urdf               | -->
-<!-- |    EDITING THIS FILE BY HAND IS NOT RECOMMENDED                                 | -->
-<!-- =================================================================================== -->
-<robot name="mobile_bot">
+<?xml version="1.0"?>
+<robot name="test_bot" xmlns:xacro="http://ros.org/wiki/xacro">
+  <!-- Define robot constants -->
+  <xacro:property name="base_width" value="0.31"/>
+  <xacro:property name="base_length" value="0.52"/>
+  <xacro:property name="base_height" value="0.18"/>
+  <xacro:property name="wheel_radius" value="0.10"/>
+  <xacro:property name="wheel_width" value="0.04"/>
+  <xacro:property name="wheel_zoff" value="0.05"/>
+  <xacro:property name="wheel_xoff" value="0.18"/>
+  <xacro:property name="caster_radius" value="${wheel_radius+wheel_zoff-(base_height/2)}"/>
+  <xacro:property name="caster_xoff" value="0.18"/>
+  <!-- Define intertial property macros  -->
+  <xacro:macro name="box_inertia" params="m w h d">
+    <inertial>
+      <origin xyz="0 0 0" rpy="0 0 0"/>
+      <mass value="${m}"/>
+      <inertia ixx="${(m/12) * (h*h + d*d)}" ixy="0.0" ixz="0.0" iyy="${(m/12) * (w*w + d*d)}" iyz="0.0" izz="${(m/12) * (w*w + h*h)}"/>
+    </inertial>
+  </xacro:macro>
+  <xacro:macro name="cylinder_inertia" params="m r h">
+    <inertial>
+      <origin xyz="0 0 0" rpy="${pi/2} 0 0"/>
+      <mass value="${m}"/>
+      <inertia ixx="${(m/12) * (3*r*r + h*h)}" ixy = "0" ixz = "0" iyy="${(m/12) * (3*r*r + h*h)}" iyz = "0" izz="${(m/2) * (r*r)}"/>
+    </inertial>
+  </xacro:macro>
+  <xacro:macro name="sphere_inertia" params="m r">
+    <inertial>
+      <mass value="${m}"/>
+      <inertia ixx="${(2/5) * m * (r*r)}" ixy="0.0" ixz="0.0" iyy="${(2/5) * m * (r*r)}" iyz="0.0" izz="${(2/5) * m * (r*r)}"/>
+    </inertial>
+  </xacro:macro>
   <!-- Robot Base -->
   <link name="base_link">
     <visual>
       <geometry>
-        <box size="0.52 0.31 0.18"/>
+        <box size="${base_length} ${base_width} ${base_height}"/>
       </geometry>
       <material name="Cyan">
@@ -17,12 +44,8 @@
     <collision>
       <geometry>
-        <box size="0.52 0.31 0.18"/>
-      </geometry>
-    </collision>
-    <inertial>
-      <origin rpy="0 0 0" xyz="0 0 0"/>
-      <mass value="5"/>
-      <inertia ixx="0.12616666666666668" ixy="0.0" ixz="0.0" iyy="0.15270833333333336" iyz="0.0" izz="0.05354166666666667"/>
-    </inertial>
+        <box size="${base_length} ${base_width} ${base_height}"/>
+      </geometry>
+    </collision>
+    <xacro:box_inertia m="5" w="${base_width}" d="${base_length}" h="${base_height}"/>
   </link>
   <!-- Robot Footprint -->
@@ -31,68 +54,41 @@
     <parent link="base_footprint"/>
     <child link="base_link"/>
-    <origin rpy="0 0 0" xyz="0 0 0.15000000000000002"/>
-  </joint>
-  <link name="drivewhl_l_link">
-    <visual>
-      <origin rpy="1.5707963267948966 0 0" xyz="0 0 0"/>
-      <geometry>
-        <cylinder length="0.04" radius="0.1"/>
-      </geometry>
-      <material name="Gray">
-        <color rgba="0.5 0.5 0.5 1.0"/>
-      </material>
-    </visual>
-    <collision>
-      <origin rpy="1.5707963267948966 0 0" xyz="0 0 0"/>
-      <geometry>
-        <cylinder length="0.04" radius="0.1"/>
-      </geometry>
-    </collision>
-    <inertial>
-      <origin rpy="1.5707963267948966 0 0" xyz="0 0 0"/>
-      <mass value="2"/>
-      <inertia ixx="0.005266666666666667" ixy="0" ixz="0" iyy="0.005266666666666667" iyz="0" izz="0.010000000000000002"/>
-    </inertial>
-  </link>
-  <joint name="drivewhl_l_joint" type="continuous">
-    <parent link="base_link"/>
-    <child link="drivewhl_l_link"/>
-    <origin rpy="0 0 0" xyz="-0.18 0.175 -0.05"/>
-    <axis xyz="0 1 0"/>
-  </joint>
-  <link name="drivewhl_r_link">
-    <visual>
-      <origin rpy="1.5707963267948966 0 0" xyz="0 0 0"/>
-      <geometry>
-        <cylinder length="0.04" radius="0.1"/>
-      </geometry>
-      <material name="Gray">
-        <color rgba="0.5 0.5 0.5 1.0"/>
-      </material>
-    </visual>
-    <collision>
-      <origin rpy="1.5707963267948966 0 0" xyz="0 0 0"/>
-      <geometry>
-        <cylinder length="0.04" radius="0.1"/>
-      </geometry>
-    </collision>
-    <inertial>
-      <origin rpy="1.5707963267948966 0 0" xyz="0 0 0"/>
-      <mass value="2"/>
-      <inertia ixx="0.005266666666666667" ixy="0" ixz="0" iyy="0.005266666666666667" iyz="0" izz="0.010000000000000002"/>
-    </inertial>
-  </link>
-  <joint name="drivewhl_r_joint" type="continuous">
-    <parent link="base_link"/>
-    <child link="drivewhl_r_link"/>
-    <origin rpy="0 0 0" xyz="-0.18 -0.175 -0.05"/>
-    <axis xyz="0 1 0"/>
-  </joint>
+    <origin xyz="0 0 ${(wheel_radius+wheel_zoff)}" rpy="0 0 0"/>
+  </joint>
+    <!-- Drive Wheels -->
+  <xacro:macro name="wheel" params="prefix x_reflect y_reflect">
+    <link name="${prefix}_link">
+      <visual>
+        <origin xyz="0 0 0" rpy="${pi/2} 0 0"/>
+        <geometry>
+            <cylinder radius="${wheel_radius}" length="${wheel_width}"/>
+        </geometry>
+        <material name="Gray">
+          <color rgba="0.5 0.5 0.5 1.0"/>
+        </material>
+      </visual>
+      <collision>
+        <origin xyz="0 0 0" rpy="${pi/2} 0 0"/>
+        <geometry>
+          <cylinder radius="${wheel_radius}" length="${wheel_width}"/>
+        </geometry>
+      </collision>
+      <xacro:cylinder_inertia m="2" r="${wheel_radius}" h="${wheel_width}"/>
+    </link>
+    <joint name="${prefix}_joint" type="continuous">
+      <parent link="base_link"/>
+      <child link="${prefix}_link"/>
+      <origin xyz="${x_reflect*wheel_xoff} ${y_reflect*((base_width/2)+(wheel_width/2))} ${-wheel_zoff}" rpy="0 0 0"/>
+      <axis xyz="0 1 0"/>
+    </joint>
+  </xacro:macro>
+  <xacro:wheel prefix="drivewhl_l" x_reflect="-1.0" y_reflect="1.0" />
+  <xacro:wheel prefix="drivewhl_r" x_reflect="-1.0" y_reflect="-1.0" />
   <!-- Caster Wheel -->
   <link name="front_caster">
     <visual>
-      <origin rpy="0 0 0" xyz="0 0 0"/>
-      <geometry>
-        <sphere radius="0.060000000000000026"/>
+      <origin xyz="0 0 0" rpy="0 0 0"/>
+      <geometry>
+        <sphere radius="${caster_radius}"/>
       </geometry>
       <material name="Cyan">
@@ -101,13 +97,10 @@
     </visual>
     <collision>
-      <origin rpy="0 0 0" xyz="0 0 0"/>
-      <geometry>
-        <sphere radius="0.060000000000000026"/>
-      </geometry>
-    </collision>
-    <inertial>
-      <mass value="2"/>
-      <inertia ixx="0.0028800000000000023" ixy="0.0" ixz="0.0" iyy="0.0028800000000000023" iyz="0.0" izz="0.0028800000000000023"/>
-    </inertial>
+      <origin xyz="0 0 0" rpy="0 0 0"/>
+      <geometry>
+        <sphere radius="${caster_radius}"/>
+      </geometry>
+    </collision>
+    <xacro:sphere_inertia m="2" r="${caster_radius}"/>
   </link>
   <gazebo reference="front_caster">
@@ -118,5 +111,5 @@
     <parent link="base_link"/>
     <child link="front_caster"/>
-    <origin rpy="0 0 0" xyz="0.18 0 -0.09"/>
+    <origin xyz="${caster_xoff} 0 ${-(base_height/2)}" rpy="0 0 0"/>
   </joint>
   <!-- Imu Plugin Set Up -->
@@ -132,9 +125,5 @@
       </geometry>
     </collision>
-    <inertial>
-      <origin rpy="0 0 0" xyz="0 0 0"/>
-      <mass value="0.1"/>
-      <inertia ixx="0.0001666666666666667" ixy="0.0" ixz="0.0" iyy="0.0001666666666666667" iyz="0.0" izz="0.0001666666666666667"/>
-    </inertial>
+    <xacro:box_inertia m="0.1" w="0.1" d="0.1" h="0.1"/>
   </link>
   <joint name="imu_joint" type="fixed">
@@ -145,5 +134,5 @@
   <gazebo reference="imu_link">
     <sensor name="imu_sensor" type="imu">
-      <plugin filename="libgazebo_ros_imu_sensor.so" name="imu_plugin">
+    <plugin filename="libgazebo_ros_imu_sensor.so" name="imu_plugin">
         <ros>
           <remapping>~/out:=imu</remapping>
@@ -211,5 +200,5 @@
   </gazebo>
   <gazebo>
-    <plugin filename="libgazebo_ros_diff_drive.so" name="diff_drive">
+    <plugin name='diff_drive' filename='libgazebo_ros_diff_drive.so'>
       <update_rate>30</update_rate>
       <!-- wheels -->
@@ -241,18 +230,18 @@
   <link name="lidar_link">
     <inertial>
-      <origin rpy="0 0 0" xyz="0 0 0"/>
+      <origin xyz="0 0 0" rpy="0 0 0"/>
       <mass value="0.125"/>
-      <inertia ixx="0.001" ixy="0" ixz="0" iyy="0.001" iyz="0" izz="0.001"/>
-    </inertial>
-    <collision>
-      <origin rpy="0 0 0" xyz="0 0 0"/>
-      <geometry>
-        <cylinder length="0.055" radius="0.0508"/>
-      </geometry>
-    </collision>
-    <visual>
-      <origin rpy="0 0 0" xyz="0 0 0"/>
-      <geometry>
-        <cylinder length="0.055" radius="0.0508"/>
+      <inertia ixx="0.001"  ixy="0"  ixz="0" iyy="0.001" iyz="0" izz="0.001" />
+    </inertial>
+    <collision>
+      <origin xyz="0 0 0" rpy="0 0 0"/>
+      <geometry>
+        <cylinder radius="0.0508" length="0.055"/>
+      </geometry>
+    </collision>
+    <visual>
+      <origin xyz="0 0 0" rpy="0 0 0"/>
+      <geometry>
+        <cylinder radius="0.0508" length="0.055"/>
       </geometry>
     </visual>
@@ -261,5 +250,5 @@
     <parent link="base_link"/>
     <child link="lidar_link"/>
-    <origin rpy="0 0 0" xyz="0 0 0.12"/>
+    <origin xyz="0 0 0.12" rpy="0 0 0"/>
   </joint>
   <gazebo reference="lidar_link">
@@ -288,5 +277,5 @@
         </noise>
       </ray>
-      <plugin filename="libgazebo_ros_ray_sensor.so" name="scan">
+      <plugin name="scan" filename="libgazebo_ros_ray_sensor.so">
         <ros>
           <remapping>~/out:=scan</remapping>
