Commit message: Finished static transform broadcaster for lidar. Changed wheel odometry and imu frame to launch parameters

File: all_launch/urdf/lidar.urdf (robot description, URDF)
Before this commit: robot ambot, 3 links, 2 joints
Links:
- removed link imu
Joints:
- removed joint imu_joint

File: all_launch/urdf/lidar.xacro (robot description, xacro)
@@ -8,9 +8,3 @@
         <origin xyz="0 0 0" rpy="0 0 ${pi/2}"/>
     </joint>
-    <link name="imu"/>
-    <joint name="imu_joint" type="fixed">
-        <parent link="base_footprint"/>
-        <child link="imu"/>
-        <origin xyz="0 0 0" rpy="0 0 0"/>
-    </joint>
 </robot>

Commit message: Fully working on raspberry pi with nav2 parameters tuned optimally

File: all_launch/urdf/lidar.urdf (robot description, URDF)
Before this commit: robot ambot, 2 links, 1 joints
Joints:
- joint laser_joint: origin xyz=0 0 0 rpy=0 0 1.5707963267948966 -> xyz=0 0 0 rpy=0 0 3.141592653589793

File: all_launch/urdf/lidar.xacro (robot description, xacro)
@@ -6,5 +6,5 @@
         <parent link="base_footprint"/>
         <child link="laser"/>
-        <origin xyz="0 0 0" rpy="0 0 ${pi/2}"/>
+        <origin xyz="0 0 0" rpy="0 0 ${pi}"/>
     </joint>
 </robot>
